File: starbie_KICAD.kicad_pcb (KiCad board)
At the start: 2 copper layers, 84.7 x 68 mm, 7 parts, among them J1 Conn_01x04_Pin, J2 Conn_01x08_Pin, SW1 SW_Push, SW2 SW_Push, U1 DHT11, U2 XIAO-ESP32-C3-SMD

Commit message: Autosave
Parts:
- moved SW2 55.9 mm to (98.5, 80.5)
- moved J2 49.4 mm to (171.5, 94.9)
Changed lines of the file:
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@@
 	(footprint "Button_Switch_Keyboard:SW_Cherry_MX_1.00u_PCB"
 		(layer "F.Cu")
-		(at 152.54 94.92)
+		(at 98.54 80.51)
 		(descr "Cherry MX keyswitch, 1.00u, PCB mount, http://cherryamericas.com/wp-content/uploads/2014/12/mx_cat.pdf")
 		(tags "Cherry MX keyswitch 1.00u PCB")
@@
 	(footprint "Connector_PinHeader_2.54mm:PinHeader_1x08_P2.54mm_Vertical"
 		(layer "F.Cu")
-		(at 212.5 122.42)
+		(at 171.5 94.88)
 		(descr "Through hole straight pin header, 1x08, 2.54mm pitch, single row")
 		(tags "Through hole pin header THT 1x08 2.54mm single row")

Commit message: Autosave
Parts:
- moved SW1 5.57 mm to (147.5, 74.5)
- moved U2 5.57 mm to (194.5, 79.6)
- moved U1 5.57 mm to (171.4, 48.9)
- moved J1 5.57 mm to (168.5, 68.0)
- moved J2 5.57 mm to (175.5, 91.0)

Commit message: Autosave
Parts:
- moved J1 60.6 mm to (141.0, 122.0)
- moved SW1 51.5 mm to (102.8, 49.0)
- moved J2 37.5 mm to (196.5, 122.1)
Changed lines of the file:
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@@
 	(footprint "Button_Switch_Keyboard:SW_Cherry_MX_1.00u_PCB"
 		(layer "F.Cu")
-		(at 147.54 74.547)
+		(at 102.85 48.96)
 		(descr "Cherry MX keyswitch, 1.00u, PCB mount, http://cherryamericas.com/wp-content/uploads/2014/12/mx_cat.pdf")
 		(tags "Cherry MX keyswitch 1.00u PCB")
@@
 	(footprint "Imported Parts:Display_128x64_096_I2C"
 		(layer "F.Cu")
-		(at 168.5 67.992)
+		(at 141 121.992)
 		(descr "Display 0.96\" OLED 128x64 pixel with SSD1306 controller and I2C interface")
 		(tags "display OLED SSD1306 128x64")
@@
 	(footprint "Connector_PinHeader_2.54mm:PinHeader_1x08_P2.54mm_Vertical"
 		(layer "F.Cu")
-		(at 175.5 91.007)
+		(at 196.5 122.11)
 		(descr "Through hole straight pin header, 1x08, 2.54mm pitch, single row")
 		(tags "Through hole pin header THT 1x08 2.54mm single row")

Commit message: Autosave
Parts:
- moved U2 35.8 mm to (223.4, 58.5)
- moved U1 22.4 mm to (171.5, 26.5)
Changed lines of the file:
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@@
 	(footprint "Imported Parts:XIAO-ESP32-C6-DIP"
 		(layer "F.Cu")
-		(at 194.5 79.627 90)
+		(at 223.38 58.5 90)
 		(property "Reference" "U2"
 			(at -0.125 -10.25 90)
@@
 	(footprint "Sensor:Aosong_DHT11_5.5x12.0_P2.54mm"
 		(layer "F.Cu")
-		(at 171.398286 48.858992)
+		(at 171.5 26.46)
 		(descr "Temperature and humidity module, http://akizukidenshi.com/download/ds/aosong/DHT11.pdf")
 		(tags "Temperature and humidity module")

Commit message: Autosave
Parts:
- moved U2 31.6 mm to (196.0, 74.3)
Other:
- board size 84.7 x 68 mm -> 93.3 x 74.9 mm

Commit message: Autosave
Parts:
- moved U1 25.9 mm to (171.5, 52.4)
Changed lines of the file:
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@@
 	(footprint "Sensor:Aosong_DHT11_5.5x12.0_P2.54mm"
 		(layer "F.Cu")
-		(at 171.5 26.46)
+		(at 171.5 52.38)
 		(descr "Temperature and humidity module, http://akizukidenshi.com/download/ds/aosong/DHT11.pdf")
 		(tags "Temperature and humidity module")

Commit message: Autosave
Parts:
- moved U1 4.60 mm to (175.2, 55.1), turned to -90 degrees
Changed lines of the file:
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@@
 	(footprint "Sensor:Aosong_DHT11_5.5x12.0_P2.54mm"
 		(layer "F.Cu")
-		(at 171.5 52.38)
+		(at 175.2125 55.0975 -90)
 		(descr "Temperature and humidity module, http://akizukidenshi.com/download/ds/aosong/DHT11.pdf")
 		(tags "Temperature and humidity module")
 		(property "Reference" "U1"
-			(at -1 -3.5 0)
+			(at -1 -3.5 90)
 			(layer "F.SilkS")
 			(effects
@@
 		)
 		(property "Value" "DHT11"
-			(at 0 11.3 0)
+			(at 0 11.3 90)
 			(layer "F.Fab")
 			(effects
@@
 		)
 		(property "Datasheet" "http://akizukidenshi.com/download/ds/aosong/DHT11.pdf"
-			(at 0 0 0)
+			(at 0 0 270)
 			(unlocked yes)
 			(layer "F.Fab")
@@
 		)
 		(property "Description" "3.3V to 5.5V, temperature and humidity module, DHT11"
-			(at 0 0 0)
+			(at 0 0 270)
 			(unlocked yes)
 			(layer "F.Fab")
@@
 		(duplicate_pad_numbers_are_jumpers no)
 		(fp_line
+			(start -2.88 9.94)
+			(end -2.88 -2.31)
+			(stroke
+				(width 0.12)
+				(type solid)
+			)
+			(layer "F.SilkS")
+		)
+		(fp_line
+			(start 2.88 9.94)
+			(end -2.88 9.94)
+			(stroke
+				(width 0.12)
+				(type solid)
+			)
+			(layer "F.SilkS")
+		)
+		(fp_line
+			(start -2.87 -2.32)
+			(end 2.87 -2.32)
+			(stroke
+				(width 0.12)
+				(type solid)
+			)
+			(layer "F.SilkS")
+		)
+		(fp_line
+			(start 2.88 -2.32)
+			(end 2.88 9.94)
+			(stroke
+				(width 0.12)
+				(type solid)
+			)
+			(layer "F.SilkS")
+		)
+		(fp_line
 			(start -3.16 -2.6)
 			(end -3.16 -0.6)
@@
 		)
 		(fp_line
-			(start -2.88 9.94)
-			(end -2.88 -2.31)
-			(stroke
-				(width 0.12)
-				(type solid)
-			)
-			(layer "F.SilkS")
-		)
-		(fp_line
-			(start -2.87 -2.32)
-			(end 2.87 -2.32)
-			(stroke
-				(width 0.12)
-				(type solid)
-			)
-			(layer "F.SilkS")
-		)
-		(fp_line
-			(start 2.88 -2.32)
-			(end 2.88 9.94)
-			(stroke
-				(width 0.12)
-				(type solid)
-			)
-			(layer "F.SilkS")
-		)
-		(fp_line
-			(start 2.88 9.94)
-			(end -2.88 9.94)
-			(stroke
-				(width 0.12)
-				(type solid)
-			)
-			(layer "F.SilkS")
+			(start -3 10.06)
+			(end -3 -2.44)
+			(stroke
+				(width 0.05)
+				(type solid)
+			)
+			(layer "F.CrtYd")
+		)
+		(fp_line
+			(start 3 10.06)
+			(end -3 10.06)
+			(stroke
+				(width 0.05)
+				(type solid)
+			)
+			(layer "F.CrtYd")
 		)
 		(fp_line
@@
 		)
 		(fp_line
-			(start -3 10.06)
-			(end -3 -2.44)
-			(stroke
-				(width 0.05)
-				(type solid)
-			)
-			(layer "F.CrtYd")
-		)
-		(fp_line
 			(start 3 -2.44)
 			(end 3 10.06)
@@
 		)
 		(fp_line
-			(start 3 10.06)
-			(end -3 10.06)
-			(stroke
-				(width 0.05)
-				(type solid)
-			)
-			(layer "F.CrtYd")
+			(start 2.75 9.81)
+			(end -2.75 9.81)
+			(stroke
+				(width 0.1)
+				(type solid)
+			)
+			(layer "F.Fab")
 		)
 		(fp_line
@@
 			(layer "F.Fab")
 		)
-		(fp_line
-			(start 2.75 9.81)
-			(end -2.75 9.81)
-			(stroke
-				(width 0.1)
-				(type solid)
-			)
-			(layer "F.Fab")
-		)
 		(fp_text user "${REFERENCE}"
-			(at 0 3.81 0)
+			(at 0 3.81 90)
 			(layer "F.Fab")
 			(effects
@@
 		)
 		(pad "1" thru_hole rect
-			(at 0 0)
+			(at 0 0 270)
 			(size 1.5 1.5)
 			(drill 0.8)
@@
 		)
 		(pad "2" thru_hole circle
-			(at 0 2.54)
+			(at 0 2.54 270)
 			(size 1.5 1.5)
 			(drill 0.8)
@@
 		)
 		(pad "3" thru_hole circle
-			(at 0 5.08)
+			(at 0 5.08 270)
 			(size 1.5 1.5)
 			(drill 0.8)
@@
 		)
 		(pad "4" thru_hole circle
-			(at 0 7.62)
-			(size 1.5 1.5)
-			(drill 0.8)
+			(at 0 7.62 270)
+			(size 1.5 1.5)
+			(drill 0.8)

Commit message: Autosave
Parts:
- moved U1 1.56 mm to (174.5, 56.5)
Changed lines of the file:
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@@
 	(footprint "Sensor:Aosong_DHT11_5.5x12.0_P2.54mm"
 		(layer "F.Cu")
-		(at 175.2125 55.0975 -90)
+		(at 174.54 56.5 -90)
 		(descr "Temperature and humidity module, http://akizukidenshi.com/download/ds/aosong/DHT11.pdf")
 		(tags "Temperature and humidity module")
