File: starbie_KICAD.kicad_pcb (KiCad board)
At the start: 2 copper layers, 99.9 x 80.2 mm, 9 parts, among them J1 Conn_01x04_Pin, J2 Conn_01x08_Pin, SW1 SW_Push, SW2 SW_Push, U1 DHT11, U2 XIAO-ESP32-C3-SMD

Commit message: Autosave
Parts:
- renumbered G*** to ?
Changed lines of the file:
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@@
 		(layer "F.Cu")
 		(at 141.941178 55.669402 -70)
-		(property "Reference" "G***"
+		(property "Reference" ""
 			(at 0 0 110)
 			(layer "F.SilkS")

Commit message: Autosave
Parts:
- renumbered G*** to ?
Changed lines of the file:
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@@
 		(layer "F.Cu")
 		(at 203.5 97.5)
-		(property "Reference" "G***"
+		(property "Reference" ""
 			(at 0 0 0)
 			(layer "F.SilkS")

Commit message: PCB Save
Parts:
- removed the ? at (141.9, 55.7)

Commit message: Autosave
Parts:
- added G***: LOGO, images:b, F.Cu at (204.5, 53.0)

Commit message: Autosave
Parts:
- renumbered G*** to ?
Changed lines of the file:
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@@
 		(layer "F.Cu")
 		(at 204.5 53)
-		(property "Reference" "G***"
+		(property "Reference" ""
 			(at 0 0 0)
 			(layer "F.SilkS")

Commit message: Autosave
Parts:
- turned ? to 20 degrees

Commit message: Autosave
Parts:
- moved ? 5.22 mm to (206.0, 58.0), turned to 30 degrees

Commit message: PCB Save
Parts:
- moved ? 0.71 mm to (205.5, 57.5)
Changed lines of the file:
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@@
 	(footprint "images:b"
 		(layer "F.Cu")
-		(at 206 58 30)
+		(at 205.5 57.5 30)
 		(property "Reference" ""
 			(at 0 0 30)
